File: hardware/ledAndDriver.sch (KiCad schematic (older format))
At the start: 4 parts, among them Q3 BSS138

Commit message: replaced separated driver parts with driver chips and LED bars
Parts:
- removed D1: LED, LED_SMD:LED_0201_0603Metric, symbol Device:LED
- removed Q3: BSS138, Package_TO_SOT_SMD:SOT-23, symbol Transistor_FET:BSS138
- removed R10: 100K, Resistor_SMD:R_0201_0603Metric, symbol Device:R
- removed R9: R, Resistor_SMD:R_0201_0603Metric, symbol Device:R
Changed lines of the file:
@@
 EESchema Schematic File Version 4
-LIBS:heating-control-cache
+LIBS:relays-device-cache
 EELAYER 30 0
 EELAYER END
@@
 Comment4 ""
 $EndDescr
-$Comp
-L Transistor_FET:BSS138 Q?
-U 1 1 5D9C9B06
-P 4300 3500
-AR Path="/5D9B8E7D/5D9C7CE9/5D9C9B06" Ref="Q?"  Part="1"
-AR Path="/5D9B8E7D/5D9F6DFE/5D9C9B06" Ref="Q3"  Part="1"
-AR Path="/5D9B8E7D/5D9F7D18/5D9C9B06" Ref="Q4"  Part="1"
-AR Path="/5D9B8E7D/5DA4749D/5D9C9B06" Ref="Q5"  Part="1"
-AR Path="/5D9B8E7D/5DA49210/5D9C9B06" Ref="Q6"  Part="1"
-AR Path="/5D9B8E7D/5DA4947F/5D9C9B06" Ref="Q7"  Part="1"
-AR Path="/5D9B8E7D/5DA496EE/5D9C9B06" Ref="Q8"  Part="1"
-AR Path="/5D9B8E7D/5DA4995D/5D9C9B06" Ref="Q9"  Part="1"
-AR Path="/5D9B8E7D/5DA49BCC/5D9C9B06" Ref="Q10"  Part="1"
-AR Path="/5D9B8E7D/5DA49F6E/5D9C9B06" Ref="Q11"  Part="1"
-AR Path="/5D9B8E7D/5DA4A1DF/5D9C9B06" Ref="Q12"  Part="1"
-AR Path="/5D9F7D18/5D9C9B06" Ref="Q4"  Part="1"
-AR Path="/5D9F6DFE/5D9C9B06" Ref="Q3"  Part="1"
-AR Path="/5DA4749D/5D9C9B06" Ref="Q5"  Part="1"
-AR Path="/5DA49210/5D9C9B06" Ref="Q6"  Part="1"
-AR Path="/5DA4947F/5D9C9B06" Ref="Q7"  Part="1"
-AR Path="/5DA496EE/5D9C9B06" Ref="Q8"  Part="1"
-AR Path="/5DA4995D/5D9C9B06" Ref="Q9"  Part="1"
-AR Path="/5DA49BCC/5D9C9B06" Ref="Q10"  Part="1"
-AR Path="/5DA49F6E/5D9C9B06" Ref="Q11"  Part="1"
-AR Path="/5DA4A1DF/5D9C9B06" Ref="Q12"  Part="1"
-AR Path="/5D9B8E7D/5DAA1288/5D9C9B06" Ref="Q13"  Part="1"
-AR Path="/5D9B8E7D/5DAA160B/5D9C9B06" Ref="Q14"  Part="1"
-AR Path="/5D9B8E7D/5DAA31F1/5D9C9B06" Ref="Q15"  Part="1"
-AR Path="/5D9B8E7D/5DAA3574/5D9C9B06" Ref="Q16"  Part="1"
-AR Path="/5D9B8E7D/5DAA38F7/5D9C9B06" Ref="Q17"  Part="1"
-AR Path="/5D9B8E7D/5DAA3C7A/5D9C9B06" Ref="Q18"  Part="1"
-F 0 "Q18" H 4506 3546 50  0000 L CNN
-F 1 "BSS138" H 4506 3455 50  0000 L CNN
-F 2 "Package_TO_SOT_SMD:SOT-23" H 4500 3425 50  0001 L CIN
-F 3 "https://www.fairchildsemi.com/datasheets/BS/BSS138.pdf" H 4300 3500 50  0001 L CNN
-	1    4300 3500
-	1    0    0    -1
-$EndComp
-$Comp
-L Device:R R?
-U 1 1 5D9C9B0C
-P 4000 3750
-AR Path="/5D9B8E7D/5D9C7CE9/5D9C9B0C" Ref="R?"  Part="1"
-AR Path="/5D9B8E7D/5D9F6DFE/5D9C9B0C" Ref="R10"  Part="1"
-AR Path="/5D9B8E7D/5D9F7D18/5D9C9B0C" Ref="R12"  Part="1"
-AR Path="/5D9B8E7D/5DA4749D/5D9C9B0C" Ref="R14"  Part="1"
-AR Path="/5D9B8E7D/5DA49210/5D9C9B0C" Ref="R16"  Part="1"
-AR Path="/5D9B8E7D/5DA4947F/5D9C9B0C" Ref="R18"  Part="1"
-AR Path="/5D9B8E7D/5DA496EE/5D9C9B0C" Ref="R20"  Part="1"
-AR Path="/5D9B8E7D/5DA4995D/5D9C9B0C" Ref="R22"  Part="1"
-AR Path="/5D9B8E7D/5DA49BCC/5D9C9B0C" Ref="R24"  Part="1"
-AR Path="/5D9B8E7D/5DA49F6E/5D9C9B0C" Ref="R26"  Part="1"
-AR Path="/5D9B8E7D/5DA4A1DF/5D9C9B0C" Ref="R28"  Part="1"
-AR Path="/5D9F7D18/5D9C9B0C" Ref="R12"  Part="1"
-AR Path="/5D9F6DFE/5D9C9B0C" Ref="R10"  Part="1"
-AR Path="/5DA4749D/5D9C9B0C" Ref="R14"  Part="1"
-AR Path="/5DA49210/5D9C9B0C" Ref="R16"  Part="1"
-AR Path="/5DA4947F/5D9C9B0C" Ref="R18"  Part="1"
-AR Path="/5DA496EE/5D9C9B0C" Ref="R20"  Part="1"
-AR Path="/5DA4995D/5D9C9B0C" Ref="R22"  Part="1"
-AR Path="/5DA49BCC/5D9C9B0C" Ref="R24"  Part="1"
-AR Path="/5DA49F6E/5D9C9B0C" Ref="R26"  Part="1"
-AR Path="/5DA4A1DF/5D9C9B0C" Ref="R28"  Part="1"
-AR Path="/5D9B8E7D/5DAA1288/5D9C9B0C" Ref="R30"  Part="1"
-AR Path="/5D9B8E7D/5DAA160B/5D9C9B0C" Ref="R32"  Part="1"
-AR Path="/5D9B8E7D/5DAA31F1/5D9C9B0C" Ref="R34"  Part="1"
-AR Path="/5D9B8E7D/5DAA3574/5D9C9B0C" Ref="R36"  Part="1"
-AR Path="/5D9B8E7D/5DAA38F7/5D9C9B0C" Ref="R38"  Part="1"
-AR Path="/5D9B8E7D/5DAA3C7A/5D9C9B0C" Ref="R40"  Part="1"
-F 0 "R40" H 4070 3796 50  0000 L CNN
-F 1 "100K" H 4070 3705 50  0000 L CNN
-F 2 "Resistor_SMD:R_0201_0603Metric" V 3930 3750 50  0001 C CNN
-F 3 "~" H 4000 3750 50  0001 C CNN
-	1    4000 3750
-	1    0    0    -1
-$EndComp
-Wire Wire Line
-	4400 3300 4400 3200
-Wire Wire Line
-	4000 3600 4000 3500
-Wire Wire Line
-	4000 3500 4100 3500
-Wire Wire Line
-	4400 3700 4400 3950
-Wire Wire Line
-	4000 3900 4000 3950
-Wire Wire Line
-	4000 3950 4400 3950
-Connection ~ 4400 3950
-Wire Wire Line
-	4400 3950 4400 4050
-Connection ~ 4000 3500
-$Comp
-L Device:R R?
-U 1 1 5D9C9B23
-P 3800 2500
-AR Path="/5D9B8E7D/5D9C7CE9/5D9C9B23" Ref="R?"  Part="1"
-AR Path="/5D9B8E7D/5D9F6DFE/5D9C9B23" Ref="R9"  Part="1"
-AR Path="/5D9B8E7D/5D9F7D18/5D9C9B23" Ref="R11"  Part="1"
-AR Path="/5D9B8E7D/5DA4749D/5D9C9B23" Ref="R13"  Part="1"
-AR Path="/5D9B8E7D/5DA49210/5D9C9B23" Ref="R15"  Part="1"
-AR Path="/5D9B8E7D/5DA4947F/5D9C9B23" Ref="R17"  Part="1"
-AR Path="/5D9B8E7D/5DA496EE/5D9C9B23" Ref="R19"  Part="1"
-AR Path="/5D9B8E7D/5DA4995D/5D9C9B23" Ref="R21"  Part="1"
-AR Path="/5D9B8E7D/5DA49BCC/5D9C9B23" Ref="R23"  Part="1"
-AR Path="/5D9B8E7D/5DA49F6E/5D9C9B23" Ref="R25"  Part="1"
-AR Path="/5D9B8E7D/5DA4A1DF/5D9C9B23" Ref="R27"  Part="1"
-AR Path="/5D9F7D18/5D9C9B23" Ref="R11"  Part="1"
-AR Path="/5D9F6DFE/5D9C9B23" Ref="R9"  Part="1"
-AR Path="/5DA4749D/5D9C9B23" Ref="R13"  Part="1"
-AR Path="/5DA49210/5D9C9B23" Ref="R15"  Part="1"
-AR Path="/5DA4947F/5D9C9B23" Ref="R17"  Part="1"
-AR Path="/5DA496EE/5D9C9B23" Ref="R19"  Part="1"
-AR Path="/5DA4995D/5D9C9B23" Ref="R21"  Part="1"
-AR Path="/5DA49BCC/5D9C9B23" Ref="R23"  Part="1"
-AR Path="/5DA49F6E/5D9C9B23" Ref="R25"  Part="1"
-AR Path="/5DA4A1DF/5D9C9B23" Ref="R27"  Part="1"
-AR Path="/5D9B8E7D/5DAA1288/5D9C9B23" Ref="R29"  Part="1"
-AR Path="/5D9B8E7D/5DAA160B/5D9C9B23" Ref="R31"  Part="1"
-AR Path="/5D9B8E7D/5DAA31F1/5D9C9B23" Ref="R33"  Part="1"
-AR Path="/5D9B8E7D/5DAA3574/5D9C9B23" Ref="R35"  Part="1"
-AR Path="/5D9B8E7D/5DAA38F7/5D9C9B23" Ref="R37"  Part="1"
-AR Path="/5D9B8E7D/5DAA3C7A/5D9C9B23" Ref="R39"  Part="1"
-F 0 "R39" H 3870 2546 50  0000 L CNN
-F 1 "R" H 3870 2455 50  0000 L CNN
-F 2 "Resistor_SMD:R_0201_0603Metric" V 3730 2500 50  0001 C CNN
-F 3 "~" H 3800 2500 50  0001 C CNN
-	1    3800 2500
-	1    0    0    -1
-$EndComp
-$Comp
-L Device:LED D?
-U 1 1 5D9C9B2F
-P 3800 2950
-AR Path="/5D9B8E7D/5D9C7CE9/5D9C9B2F" Ref="D?"  Part="1"
-AR Path="/5D9B8E7D/5D9F6DFE/5D9C9B2F" Ref="D1"  Part="1"
-AR Path="/5D9B8E7D/5D9F7D18/5D9C9B2F" Ref="D2"  Part="1"
-AR Path="/5D9B8E7D/5DA4749D/5D9C9B2F" Ref="D4"  Part="1"
-AR Path="/5D9B8E7D/5DA49210/5D9C9B2F" Ref="D5"  Part="1"
-AR Path="/5D9B8E7D/5DA4947F/5D9C9B2F" Ref="D6"  Part="1"
-AR Path="/5D9B8E7D/5DA496EE/5D9C9B2F" Ref="D7"  Part="1"
-AR Path="/5D9B8E7D/5DA4995D/5D9C9B2F" Ref="D8"  Part="1"
-AR Path="/5D9B8E7D/5DA49BCC/5D9C9B2F" Ref="D9"  Part="1"
-AR Path="/5D9B8E7D/5DA49F6E/5D9C9B2F" Ref="D10"  Part="1"
-AR Path="/5D9B8E7D/5DA4A1DF/5D9C9B2F" Ref="D11"  Part="1"
-AR Path="/5D9F7D18/5D9C9B2F" Ref="D2"  Part="1"
-AR Path="/5D9F6DFE/5D9C9B2F" Ref="D1"  Part="1"
-AR Path="/5DA4749D/5D9C9B2F" Ref="D3"  Part="1"
-AR Path="/5DA49210/5D9C9B2F" Ref="D4"  Part="1"
-AR Path="/5DA4947F/5D9C9B2F" Ref="D5"  Part="1"
-AR Path="/5DA496EE/5D9C9B2F" Ref="D6"  Part="1"
-AR Path="/5DA4995D/5D9C9B2F" Ref="D7"  Part="1"
-AR Path="/5DA49BCC/5D9C9B2F" Ref="D8"  Part="1"
-AR Path="/5DA49F6E/5D9C9B2F" Ref="D9"  Part="1"
-AR Path="/5DA4A1DF/5D9C9B2F" Ref="D10"  Part="1"
-AR Path="/5D9B8E7D/5DAA1288/5D9C9B2F" Ref="D12"  Part="1"
-AR Path="/5D9B8E7D/5DAA160B/5D9C9B2F" Ref="D13"  Part="1"
-AR Path="/5D9B8E7D/5DAA31F1/5D9C9B2F" Ref="D14"  Part="1"
-AR Path="/5D9B8E7D/5DAA3574/5D9C9B2F" Ref="D15"  Part="1"
-AR Path="/5D9B8E7D/5DAA38F7/5D9C9B2F" Ref="D16"  Part="1"
-AR Path="/5D9B8E7D/5DAA3C7A/5D9C9B2F" Ref="D17"  Part="1"
-F 0 "D17" V 3839 2833 50  0000 R CNN
-F 1 "LED" V 3748 2833 50  0000 R CNN
-F 2 "LED_SMD:LED_0201_0603Metric" H 3800 2950 50  0001 C CNN
-F 3 "~" H 3800 2950 50  0001 C CNN
-	1    3800 2950
-	0    -1   -1   0
-$EndComp
-Wire Wire Line
-	3800 3100 3800 3200
-Wire Wire Line
-	3800 3200 4400 3200
-Wire Wire Line
-	3800 2800 3800 2650
-Wire Wire Line
-	3800 2350 3800 2250
-Connection ~ 4400 3200
-Text HLabel 3150 3500 0    50   UnSpc ~ 0
-in
-Wire Wire Line
-	3150 3500 4000 3500
-Text HLabel 5300 2800 2    50   UnSpc ~ 0
-load
-Wire Wire Line
-	4400 2800 5300 2800
-Wire Wire Line
-	4400 2800 4400 3200
-Text GLabel 3800 2250 1    50   UnSpc ~ 0
-upper3.3V
-Text GLabel 4400 4050 3    50   UnSpc ~ 0
-upperGND
 $EndSCHEMATC
