File: hardware/relais.sch (KiCad schematic (older format))
At the start: 2 parts, among them K2 FINDER-34.51

Commit message: finished schematic mostly
started to create lower PCB
Connections:
- net labels added: sw, sw2
- wire segments 8 -> 10
- no-connect marks 3 -> 1
Changed lines of the file:
@@
 EESchema Schematic File Version 4
-LIBS:relays-device-cache
+LIBS:lowerBoard-cache
 EELAYER 30 0
 EELAYER END
 $Descr A4 11693 8268
 encoding utf-8
-Sheet 4 5
+Sheet 3 17
 Title ""
 Date ""
@@
 $EndDescr
 $Comp
-L Relay:FINDER-34.51 K?
+L Relay:FINDER-34.51 K2
 U 1 1 5D9EAB55
 P 3400 1800
-AR Path="/5D9EAB55" Ref="K?"  Part="1"
-AR Path="/5D9FF064/5D9EAB55" Ref="K?"  Part="1"
-AR Path="/5D9FF064/5D9EA18F/5D9EAB55" Ref="K2"  Part="1"
-AR Path="/5D9FF064/5D9F100B/5D9EAB55" Ref="K1"  Part="1"
-F 0 "K2" H 3830 1846 50  0000 L CNN
+AR Path="/5D9F100B/5D9EAB55" Ref="K2"  Part="1"
+AR Path="/5D9EA18F/5D9EAB55" Ref="K1"  Part="1"
+AR Path="/5DABD32F/5D9EAB55" Ref="K3"  Part="1"
+AR Path="/5DABF648/5D9EAB55" Ref="K4"  Part="1"
+AR Path="/5DAC46C4/5D9EAB55" Ref="K5"  Part="1"
+AR Path="/5DADB7CB/5D9EAB55" Ref="K6"  Part="1"
+AR Path="/5DADBF91/5D9EAB55" Ref="K7"  Part="1"
+AR Path="/5DADC0EC/5D9EAB55" Ref="K8"  Part="1"
+AR Path="/5DB2249A/5D9EAB55" Ref="K9"  Part="1"
+AR Path="/5DB2252F/5D9EAB55" Ref="K10"  Part="1"
+AR Path="/5DB225BE/5D9EAB55" Ref="K11"  Part="1"
+AR Path="/5DB2264D/5D9EAB55" Ref="K12"  Part="1"
+AR Path="/5DB2271B/5D9EAB55" Ref="K13"  Part="1"
+AR Path="/5DB2283A/5D9EAB55" Ref="K14"  Part="1"
+AR Path="/5DB228C9/5D9EAB55" Ref="K15"  Part="1"
+AR Path="/5DB227AA/5D9EAB55" Ref="K16"  Part="1"
+F 0 "K16" H 3830 1846 50  0000 L CNN
 F 1 "FINDER-34.51" H 3830 1755 50  0000 L CNN
 F 2 "Relay_THT:Relay_SPDT_Finder_34.51_Vertical" H 4540 1760 50  0001 C CNN
@@
 $EndComp
 $Comp
-L Diode:1N4148 D?
+L Diode:1N4148 D2
 U 1 1 5D9EAB5B
 P 2750 1800
-AR Path="/5D9EAB5B" Ref="D?"  Part="1"
-AR Path="/5D9FF064/5D9EAB5B" Ref="D?"  Part="1"
-AR Path="/5D9FF064/5D9EA18F/5D9EAB5B" Ref="D2"  Part="1"
-AR Path="/5D9FF064/5D9F100B/5D9EAB5B" Ref="D1"  Part="1"
-F 0 "D2" V 2704 1879 50  0000 L CNN
+AR Path="/5D9F100B/5D9EAB5B" Ref="D2"  Part="1"
+AR Path="/5D9EA18F/5D9EAB5B" Ref="D1"  Part="1"
+AR Path="/5DABD32F/5D9EAB5B" Ref="D3"  Part="1"
+AR Path="/5DABF648/5D9EAB5B" Ref="D4"  Part="1"
+AR Path="/5DAC46C4/5D9EAB5B" Ref="D5"  Part="1"
+AR Path="/5DADB7CB/5D9EAB5B" Ref="D6"  Part="1"
+AR Path="/5DADBF91/5D9EAB5B" Ref="D7"  Part="1"
+AR Path="/5DADC0EC/5D9EAB5B" Ref="D8"  Part="1"
+AR Path="/5DB2249A/5D9EAB5B" Ref="D9"  Part="1"
+AR Path="/5DB2252F/5D9EAB5B" Ref="D10"  Part="1"
+AR Path="/5DB225BE/5D9EAB5B" Ref="D11"  Part="1"
+AR Path="/5DB2264D/5D9EAB5B" Ref="D12"  Part="1"
+AR Path="/5DB2271B/5D9EAB5B" Ref="D13"  Part="1"
+AR Path="/5DB2283A/5D9EAB5B" Ref="D14"  Part="1"
+AR Path="/5DB228C9/5D9EAB5B" Ref="D15"  Part="1"
+AR Path="/5DB227AA/5D9EAB5B" Ref="D16"  Part="1"
+F 0 "D16" V 2704 1879 50  0000 L CNN
 F 1 "1N4148" V 2795 1879 50  0000 L CNN
 F 2 "Diode_THT:D_DO-35_SOD27_P7.62mm_Horizontal" H 2750 1625 50  0001 C CNN
@@
 	3200 2200 3200 2100
 NoConn ~ 3500 1500
-NoConn ~ 3700 1500
-NoConn ~ 3600 2100
 Wire Wire Line
 	3200 1300 3200 1400
@@
 Text HLabel 3200 2600 3    50   UnSpc ~ 0
 in
+Text HLabel 3600 2600 3    50   UnSpc ~ 0
+sw
+Wire Wire Line
+	3600 2600 3600 2100
+Text HLabel 3700 1300 1    50   UnSpc ~ 0
+sw2
+Wire Wire Line
+	3700 1500 3700 1300
 $EndSCHEMATC

Commit message: replaced MCP23016 with MCP23017
Changed lines of the file:
@@
 $Descr A4 11693 8268
 encoding utf-8
-Sheet 3 19
+Sheet 18 19
 Title ""
 Date ""
@@
 AR Path="/5DB228C9/5D9EAB55" Ref="K15"  Part="1"
 AR Path="/5DB227AA/5D9EAB55" Ref="K16"  Part="1"
-F 0 "K16" H 3830 1846 50  0000 L CNN
+AR Path="/5D9FF064/5D9F100B/5D9EAB55" Ref="K2"  Part="1"
+AR Path="/5D9FF064/5D9EA18F/5D9EAB55" Ref="K1"  Part="1"
+AR Path="/5D9FF064/5DABD32F/5D9EAB55" Ref="K3"  Part="1"
+AR Path="/5D9FF064/5DABF648/5D9EAB55" Ref="K4"  Part="1"
+AR Path="/5D9FF064/5DAC46C4/5D9EAB55" Ref="K5"  Part="1"
+AR Path="/5D9FF064/5DADB7CB/5D9EAB55" Ref="K6"  Part="1"
+AR Path="/5D9FF064/5DADBF91/5D9EAB55" Ref="K7"  Part="1"
+AR Path="/5D9FF064/5DADC0EC/5D9EAB55" Ref="K8"  Part="1"
+AR Path="/5D9FF064/5DB2249A/5D9EAB55" Ref="K9"  Part="1"
+AR Path="/5D9FF064/5DB2252F/5D9EAB55" Ref="K10"  Part="1"
+AR Path="/5D9FF064/5DB225BE/5D9EAB55" Ref="K11"  Part="1"
+AR Path="/5D9FF064/5DB2264D/5D9EAB55" Ref="K12"  Part="1"
+AR Path="/5D9FF064/5DB2271B/5D9EAB55" Ref="K13"  Part="1"
+AR Path="/5D9FF064/5DB2283A/5D9EAB55" Ref="K15"  Part="1"
+AR Path="/5D9FF064/5DB228C9/5D9EAB55" Ref="K16"  Part="1"
+AR Path="/5D9FF064/5DB227AA/5D9EAB55" Ref="K14"  Part="1"
+F 0 "K14" H 3830 1846 50  0000 L CNN
 F 1 "FINDER-34.51" H 3830 1755 50  0000 L CNN
 F 2 "Relay_THT:Relay_SPDT_Finder_34.51_Vertical" H 4540 1760 50  0001 C CNN
@@
 AR Path="/5DB228C9/5D9EAB5B" Ref="D15"  Part="1"
 AR Path="/5DB227AA/5D9EAB5B" Ref="D16"  Part="1"
-F 0 "D16" V 2704 1879 50  0000 L CNN
+AR Path="/5D9FF064/5D9F100B/5D9EAB5B" Ref="D2"  Part="1"
+AR Path="/5D9FF064/5D9EA18F/5D9EAB5B" Ref="D1"  Part="1"
+AR Path="/5D9FF064/5DABD32F/5D9EAB5B" Ref="D3"  Part="1"
+AR Path="/5D9FF064/5DABF648/5D9EAB5B" Ref="D4"  Part="1"
+AR Path="/5D9FF064/5DAC46C4/5D9EAB5B" Ref="D5"  Part="1"
+AR Path="/5D9FF064/5DADB7CB/5D9EAB5B" Ref="D6"  Part="1"
+AR Path="/5D9FF064/5DADBF91/5D9EAB5B" Ref="D7"  Part="1"
+AR Path="/5D9FF064/5DADC0EC/5D9EAB5B" Ref="D8"  Part="1"
+AR Path="/5D9FF064/5DB2249A/5D9EAB5B" Ref="D9"  Part="1"
+AR Path="/5D9FF064/5DB2252F/5D9EAB5B" Ref="D10"  Part="1"
+AR Path="/5D9FF064/5DB225BE/5D9EAB5B" Ref="D11"  Part="1"
+AR Path="/5D9FF064/5DB2264D/5D9EAB5B" Ref="D12"  Part="1"
+AR Path="/5D9FF064/5DB2271B/5D9EAB5B" Ref="D13"  Part="1"
+AR Path="/5D9FF064/5DB2283A/5D9EAB5B" Ref="D15"  Part="1"
+AR Path="/5D9FF064/5DB228C9/5D9EAB5B" Ref="D16"  Part="1"
+AR Path="/5D9FF064/5DB227AA/5D9EAB5B" Ref="D14"  Part="1"
+F 0 "D14" V 2704 1879 50  0000 L CNN
 F 1 "1N4148" V 2795 1879 50  0000 L CNN
 F 2 "Diode_THT:D_DO-35_SOD27_P7.62mm_Horizontal" H 2750 1625 50  0001 C CNN

Commit message: lower board fixes and started with upper printed circuit board
Parts:
- K2: value FINDER-34.51 -> FINDER-43.41; footprint Relay_THT:Relay_SPDT_Finder_34.51_Vertical -> Relay_THT:Relay_SPDT_Finder_40.51
Connections:
- net labels added: GND
- net labels removed: 12V
Changed lines of the file:
@@
 $Descr A4 11693 8268
 encoding utf-8
-Sheet 18 19
+Sheet 5 19
 Title ""
 Date ""
@@
 AR Path="/5D9FF064/5DB228C9/5D9EAB55" Ref="K16"  Part="1"
 AR Path="/5D9FF064/5DB227AA/5D9EAB55" Ref="K14"  Part="1"
-F 0 "K14" H 3830 1846 50  0000 L CNN
-F 1 "FINDER-34.51" H 3830 1755 50  0000 L CNN
-F 2 "Relay_THT:Relay_SPDT_Finder_34.51_Vertical" H 4540 1760 50  0001 C CNN
+F 0 "K1" H 3830 1846 50  0000 L CNN
+F 1 "FINDER-43.41" H 3830 1755 50  0000 L CNN
+F 2 "Relay_THT:Relay_SPDT_Finder_40.51" H 4540 1760 50  0001 C CNN
 F 3 "https://gfinder.findernet.com/public/attachments/34/EN/S34USAEN.pdf" H 3400 1800 50  0001 C CNN
 	1    3400 1800
@@
 AR Path="/5D9FF064/5DB228C9/5D9EAB5B" Ref="D16"  Part="1"
 AR Path="/5D9FF064/5DB227AA/5D9EAB5B" Ref="D14"  Part="1"
-F 0 "D14" V 2704 1879 50  0000 L CNN
+F 0 "D1" V 2704 1879 50  0000 L CNN
 F 1 "1N4148" V 2795 1879 50  0000 L CNN
 F 2 "Diode_THT:D_DO-35_SOD27_P7.62mm_Horizontal" H 2750 1625 50  0001 C CNN
@@
 	3200 2200 3200 2600
 Text HLabel 3200 1300 1    50   UnSpc ~ 0
-12V
-Text HLabel 3200 2600 3    50   UnSpc ~ 0
 in
-Text HLabel 3600 2600 3    50   UnSpc ~ 0
+Text HLabel 3700 1300 1    50   UnSpc ~ 0
 sw
 Wire Wire Line
 	3600 2600 3600 2100
-Text HLabel 3700 1300 1    50   UnSpc ~ 0
+Text HLabel 3600 2600 3    50   UnSpc ~ 0
 sw2
 Wire Wire Line
 	3700 1500 3700 1300
+Text HLabel 3200 2600 3    50   UnSpc ~ 0
+GND
 $EndSCHEMATC

Commit message: continue to design lower pcb
Parts:
- removed K2: FINDER-43.41, Relay_THT:Relay_SPDT_Finder_40.51, symbol Relay:FINDER-34.51
- added U7: FINDER-43.41, Finder:FINDER-43.41, symbol Finder_43.41:FINDER-43.41
Changed lines of the file:
@@
 $Descr A4 11693 8268
 encoding utf-8
-Sheet 5 19
+Sheet 16 17
 Title ""
 Date ""
@@
 Comment4 ""
 $EndDescr
-$Comp
-L Relay:FINDER-34.51 K2
-U 1 1 5D9EAB55
-P 3400 1800
-AR Path="/5D9F100B/5D9EAB55" Ref="K2"  Part="1"
-AR Path="/5D9EA18F/5D9EAB55" Ref="K1"  Part="1"
-AR Path="/5DABD32F/5D9EAB55" Ref="K3"  Part="1"
-AR Path="/5DABF648/5D9EAB55" Ref="K4"  Part="1"
-AR Path="/5DAC46C4/5D9EAB55" Ref="K5"  Part="1"
-AR Path="/5DADB7CB/5D9EAB55" Ref="K6"  Part="1"
-AR Path="/5DADBF91/5D9EAB55" Ref="K7"  Part="1"
-AR Path="/5DADC0EC/5D9EAB55" Ref="K8"  Part="1"
-AR Path="/5DB2249A/5D9EAB55" Ref="K9"  Part="1"
-AR Path="/5DB2252F/5D9EAB55" Ref="K10"  Part="1"
-AR Path="/5DB225BE/5D9EAB55" Ref="K11"  Part="1"
-AR Path="/5DB2264D/5D9EAB55" Ref="K12"  Part="1"
-AR Path="/5DB2271B/5D9EAB55" Ref="K13"  Part="1"
-AR Path="/5DB2283A/5D9EAB55" Ref="K14"  Part="1"
-AR Path="/5DB228C9/5D9EAB55" Ref="K15"  Part="1"
-AR Path="/5DB227AA/5D9EAB55" Ref="K16"  Part="1"
-AR Path="/5D9FF064/5D9F100B/5D9EAB55" Ref="K2"  Part="1"
-AR Path="/5D9FF064/5D9EA18F/5D9EAB55" Ref="K1"  Part="1"
-AR Path="/5D9FF064/5DABD32F/5D9EAB55" Ref="K3"  Part="1"
-AR Path="/5D9FF064/5DABF648/5D9EAB55" Ref="K4"  Part="1"
-AR Path="/5D9FF064/5DAC46C4/5D9EAB55" Ref="K5"  Part="1"
-AR Path="/5D9FF064/5DADB7CB/5D9EAB55" Ref="K6"  Part="1"
-AR Path="/5D9FF064/5DADBF91/5D9EAB55" Ref="K7"  Part="1"
-AR Path="/5D9FF064/5DADC0EC/5D9EAB55" Ref="K8"  Part="1"
-AR Path="/5D9FF064/5DB2249A/5D9EAB55" Ref="K9"  Part="1"
-AR Path="/5D9FF064/5DB2252F/5D9EAB55" Ref="K10"  Part="1"
-AR Path="/5D9FF064/5DB225BE/5D9EAB55" Ref="K11"  Part="1"
-AR Path="/5D9FF064/5DB2264D/5D9EAB55" Ref="K12"  Part="1"
-AR Path="/5D9FF064/5DB2271B/5D9EAB55" Ref="K13"  Part="1"
-AR Path="/5D9FF064/5DB2283A/5D9EAB55" Ref="K15"  Part="1"
-AR Path="/5D9FF064/5DB228C9/5D9EAB55" Ref="K16"  Part="1"
-AR Path="/5D9FF064/5DB227AA/5D9EAB55" Ref="K14"  Part="1"
-F 0 "K1" H 3830 1846 50  0000 L CNN
-F 1 "FINDER-43.41" H 3830 1755 50  0000 L CNN
-F 2 "Relay_THT:Relay_SPDT_Finder_40.51" H 4540 1760 50  0001 C CNN
-F 3 "https://gfinder.findernet.com/public/attachments/34/EN/S34USAEN.pdf" H 3400 1800 50  0001 C CNN
-	1    3400 1800
-	1    0    0    -1
-$EndComp
 $Comp
 L Diode:1N4148 D2
@@
 AR Path="/5D9FF064/5DB228C9/5D9EAB5B" Ref="D16"  Part="1"
 AR Path="/5D9FF064/5DB227AA/5D9EAB5B" Ref="D14"  Part="1"
-F 0 "D1" V 2704 1879 50  0000 L CNN
+F 0 "D15" V 2704 1879 50  0000 L CNN
 F 1 "1N4148" V 2795 1879 50  0000 L CNN
 F 2 "Diode_THT:D_DO-35_SOD27_P7.62mm_Horizontal" H 2750 1625 50  0001 C CNN
@@
 	0    1    1    0
 $EndComp
-Wire Wire Line
-	3200 1500 3200 1400
 Wire Wire Line
 	2750 1650 2750 1400
@@
 	2750 2200 3200 2200
 Connection ~ 3200 2200
-Wire Wire Line
-	3200 2200 3200 2100
-NoConn ~ 3500 1500
+NoConn ~ 3600 2000
 Wire Wire Line
 	3200 1300 3200 1400
@@
 Text HLabel 3200 1300 1    50   UnSpc ~ 0
 in
-Text HLabel 3700 1300 1    50   UnSpc ~ 0
+Text HLabel 4000 2200 3    50   UnSpc ~ 0
 sw
 Wire Wire Line
-	3600 2600 3600 2100
-Text HLabel 3600 2600 3    50   UnSpc ~ 0
+	3800 1200 3800 1700
+Text HLabel 3800 1200 1    50   UnSpc ~ 0
 sw2
 Wire Wire Line
-	3700 1500 3700 1300
+	4000 2000 4000 2200
 Text HLabel 3200 2600 3    50   UnSpc ~ 0
 GND
+Wire Wire Line
+	3200 1400 3200 1600
+Wire Wire Line
+	3200 2000 3200 2200
+$Comp
+L Finder_43.41:FINDER-43.41 U7
+U 1 1 603CF29B
+P 3500 1800
+AR Path="/5D9FF064/5D9EA18F/603CF29B" Ref="U7"  Part="1"
+AR Path="/5D9FF064/5D9F100B/603CF29B" Ref="U6"  Part="1"
+AR Path="/5D9FF064/5DABD32F/603CF29B" Ref="U8"  Part="1"
+AR Path="/5D9FF064/5DABF648/603CF29B" Ref="U9"  Part="1"
+AR Path="/5D9FF064/5DAC46C4/603CF29B" Ref="U10"  Part="1"
+AR Path="/5D9FF064/5DADB7CB/603CF29B" Ref="U11"  Part="1"
+AR Path="/5D9FF064/5DADBF91/603CF29B" Ref="U12"  Part="1"
+AR Path="/5D9FF064/5DADC0EC/603CF29B" Ref="U13"  Part="1"
+AR Path="/5D9FF064/5DB2249A/603CF29B" Ref="U14"  Part="1"
+AR Path="/5D9FF064/5DB2252F/603CF29B" Ref="U15"  Part="1"
+AR Path="/5D9FF064/5DB225BE/603CF29B" Ref="U16"  Part="1"
+AR Path="/5D9FF064/5DB2264D/603CF29B" Ref="U17"  Part="1"
+AR Path="/5D9FF064/5DB2271B/603CF29B" Ref="U18"  Part="1"
+AR Path="/5D9FF064/5DB2283A/603CF29B" Ref="U19"  Part="1"
+AR Path="/5D9FF064/5DB228C9/603CF29B" Ref="U20"  Part="1"
+AR Path="/5D9FF064/5DB227AA/603CF29B" Ref="U21"  Part="1"
+AR Path="/5D9EA18F/603CF29B" Ref="U6"  Part="1"
+AR Path="/5D9F100B/603CF29B" Ref="U7"  Part="1"
+AR Path="/5DB228C9/603CF29B" Ref="U21"  Part="1"
+AR Path="/5DABD32F/603CF29B" Ref="U8"  Part="1"
+AR Path="/5DABF648/603CF29B" Ref="U9"  Part="1"
+AR Path="/5DAC46C4/603CF29B" Ref="U10"  Part="1"
+AR Path="/5DADB7CB/603CF29B" Ref="U11"  Part="1"
+AR Path="/5DADBF91/603CF29B" Ref="U12"  Part="1"
+AR Path="/5DADC0EC/603CF29B" Ref="U13"  Part="1"
+AR Path="/5DB2249A/603CF29B" Ref="U14"  Part="1"
+AR Path="/5DB2252F/603CF29B" Ref="U15"  Part="1"
+AR Path="/5DB225BE/603CF29B" Ref="U16"  Part="1"
+AR Path="/5DB2264D/603CF29B" Ref="U17"  Part="1"
+AR Path="/5DB2271B/603CF29B" Ref="U18"  Part="1"
+AR Path="/5DB2283A/603CF29B" Ref="U20"  Part="1"
+AR Path="/5DB227AA/603CF29B" Ref="U19"  Part="1"
+F 0 "U21" H 4076 1846 50  0000 L CNN
+F 1 "FINDER-43.41" H 4076 1755 50  0000 L CNN
+F 2 "Finder:FINDER-43.41" H 3050 1700 50  0001 L BNN
+F 3 "" H 3400 1800 50  0001 L BNN
+	1    3500 1800
+	1    0    0    -1
+$EndComp
 $EndSCHEMATC

Commit message: move on to 16A relays
Parts:
- U7: footprint Finder:FINDER-43.41 -> Finder:finder-43.41; symbol Finder_43.41:FINDER-43.41 -> relays-device-rescue:FINDER-43.41-Finder_43.41
Changed lines of the file:
@@
 $Descr A4 11693 8268
 encoding utf-8
-Sheet 16 17
+Sheet 3 19
 Title ""
 Date ""
@@
 AR Path="/5D9FF064/5DB228C9/5D9EAB5B" Ref="D16"  Part="1"
 AR Path="/5D9FF064/5DB227AA/5D9EAB5B" Ref="D14"  Part="1"
-F 0 "D15" V 2704 1879 50  0000 L CNN
+F 0 "D16" V 2704 1879 50  0000 L CNN
 F 1 "1N4148" V 2795 1879 50  0000 L CNN
 F 2 "Diode_THT:D_DO-35_SOD27_P7.62mm_Horizontal" H 2750 1625 50  0001 C CNN
@@
 	3200 2000 3200 2200
 $Comp
-L Finder_43.41:FINDER-43.41 U7
+L relays-device-rescue:FINDER-43.41-Finder_43.41 U7
 U 1 1 603CF29B
 P 3500 1800
@@
 AR Path="/5DB2283A/603CF29B" Ref="U20"  Part="1"
 AR Path="/5DB227AA/603CF29B" Ref="U19"  Part="1"
-F 0 "U21" H 4076 1846 50  0000 L CNN
+AR Path="/603CF29B" Ref="U21"  Part="1"
+F 0 "U19" H 4076 1846 50  0000 L CNN
 F 1 "FINDER-43.41" H 4076 1755 50  0000 L CNN
-F 2 "Finder:FINDER-43.41" H 3050 1700 50  0001 L BNN
+F 2 "Finder:finder-43.41" H 3050 1700 50  0001 L BNN
 F 3 "" H 3400 1800 50  0001 L BNN
 	1    3500 1800
